File: nissan-wbo/nissan-wbo.kicad_sch (KiCad schematic)
At the start: 26 parts, among them J1 Conn_01x02, J2 Conn_01x03, U1 MCP6004

Commit message: LCSC
Parts:
- added C4: 100n, Capacitor_SMD:C_0603_1608Metric, symbol Device:C
- C1, C8: footprint Capacitor_SMD:C_0402_1005Metric -> Capacitor_SMD:C_0603_1608Metric; LCSC (none) -> C57112
- C2, C3: LCSC (none) -> C15195
- C5, C6, C7: LCSC (none) -> C1585
- R1: LCSC (none) -> C25079
- R10, R11: LCSC (none) -> C25792
- R12, R15, R16, R17, R18, R2, R3, R6, R7: LCSC (none) -> C11702
- R13, R14: LCSC (none) -> C25744
- R8: footprint Resistor_SMD:R_0402_1005Metric -> Resistor_SMD:R_0603_1608Metric; LCSC (none) -> C4177
- R9: LCSC (none) -> C227316
- U1: LCSC (none) -> C50282
Connections:
- net GND: now also C4.1
- net at J2.2 (Pin_2), R12.2: now also C4.2
